File: electronics/alarmclock.kicad_sch (KiCad schematic)
At the start: 41 parts, among them J1 Conn_01x02, J2 SWD, J3 SocketTop, J4 SocketBottem, J5 Conn_01x02, J6 Conn_01x05, J7 Conn_01x05, J8 RotaryEncoder, Q1 Backpower, SW2 Reset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

Commit message: Changed the pcblayout after learning more about ground
Parts:
- removed Y1: 24MHz, Crystal:Crystal_SMD_SeikoEpson_MC146-4Pin_6.7x1.5mm_HandSoldering, symbol Device:Crystal_GND24
- added Y2: 32.768khz, Crystal:Crystal_SMD_3215-2Pin_3.2x1.5mm, symbol Device:Crystal
Connections:
- net OSC_IN: now also Y2.1
- net OSC_OUT: now also Y2.2
Changed lines of the file:
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@@
   (junction (at 46.99 39.37) (diameter 0) (color 0 0 0 0)
   )
-  (junction (at 85.09 127) (diameter 0) (color 0 0 0 0)
-  )
   (junction (at 35.56 30.48) (diameter 0) (color 0 0 0 0)
   )
@@
   (junction (at 72.39 146.05) (diameter 0) (color 0 0 0 0)
   )
+  (junction (at 80.01 120.65) (diameter 0) (color 0 0 0 0)
+  )
   (junction (at 80.01 137.16) (diameter 0) (color 0 0 0 0)
   )
-  (junction (at 80.01 120.65) (diameter 0) (color 0 0 0 0)
-  )
   (junction (at 118.11 101.6) (diameter 0) (color 0 0 0 0)
   )
@@
   )
   (junction (at 58.42 39.37) (diameter 0) (color 0 0 0 0)
-  )
-  (junction (at 91.44 127) (diameter 0) (color 0 0 0 0)
   )
   (junction (at 43.18 39.37) (diameter 0) (color 0 0 0 0)
@@
     (stroke (width 0) (type default))
   )
-  (wire (pts (xy 85.09 132.08) (xy 85.09 127))
-    (stroke (width 0) (type default))
-  )
   (wire (pts (xy 205.74 109.22) (xy 220.98 109.22))
     (stroke (width 0) (type default))
@@
     (stroke (width 0) (type default))
   )
-  (wire (pts (xy 80.01 123.19) (xy 80.01 120.65))
-    (stroke (width 0) (type default))
-  )
   (wire (pts (xy 187.96 119.38) (xy 189.23 119.38))
     (stroke (width 0) (type default))
@@
     (stroke (width 0) (type default))
   )
+  (wire (pts (xy 80.01 132.08) (xy 80.01 137.16))
+    (stroke (width 0) (type default))
+  )
   (polyline (pts (xy 209.55 13.97) (xy 209.55 67.31))
     (stroke (width 0) (type default))
@@
     (stroke (width 0) (type default))
   )
-  (wire (pts (xy 85.09 127) (xy 91.44 127))
-    (stroke (width 0) (type default))
-  )
   (polyline (pts (xy 222.25 148.59) (xy 273.05 148.59))
     (stroke (width 0) (type default))
@@
     (stroke (width 0) (type default))
   )
-  (wire (pts (xy 80.01 130.81) (xy 80.01 137.16))
-    (stroke (width 0) (type default))
-  )
   (wire (pts (xy 72.39 156.21) (xy 66.04 156.21))
     (stroke (width 0) (type default))
@@
     (stroke (width 0) (type default))
   )
-  (wire (pts (xy 85.09 137.16) (xy 80.01 137.16))
-    (stroke (width 0) (type default))
-  )
   (wire (pts (xy 118.11 95.25) (xy 118.11 93.98))
     (stroke (width 0) (type default))
@@
     (stroke (width 0) (type default))
   )
+  (wire (pts (xy 80.01 137.16) (xy 85.09 137.16))
+    (stroke (width 0) (type default))
+  )
   (wire (pts (xy 148.59 33.02) (xy 149.86 33.02))
     (stroke (width 0) (type default))
@@
     (stroke (width 0) (type default))
   )
-  (wire (pts (xy 74.93 132.08) (xy 85.09 132.08))
-    (stroke (width 0) (type default))
-  )
   (wire (pts (xy 205.74 107.95) (xy 205.74 109.22))
     (stroke (width 0) (type default))
@@
     (stroke (width 0) (type default))
   )
+  (wire (pts (xy 80.01 120.65) (xy 80.01 124.46))
+    (stroke (width 0) (type default))
+  )
   (wire (pts (xy 105.41 30.48) (xy 105.41 26.67))
     (stroke (width 0) (type default))
@@
     (stroke (width 0) (type default))
   )
-  (wire (pts (xy 91.44 127) (xy 91.44 137.16))
-    (stroke (width 0) (type default))
-  )
   (wire (pts (xy 35.56 30.48) (xy 43.18 30.48))
     (stroke (width 0) (type default))
@@
     (stroke (width 0) (type default))
   )
-  (wire (pts (xy 74.93 127) (xy 74.93 132.08))
-    (stroke (width 0) (type default))
-  )
   (wire (pts (xy 54.61 69.85) (xy 54.61 68.58))
     (stroke (width 0) (type default))
@@
     (stroke (width 0) (type default))
   )
-  (wire (pts (xy 91.44 120.65) (xy 91.44 127))
+  (wire (pts (xy 91.44 120.65) (xy 91.44 137.16))
     (stroke (width 0) (type default))
   )
@@
         (path "/fcd099cf-d7c6-418d-b6d0-a7fbd5aabc64"
           (reference "C7") (unit 1)
-        )
-      )
-    )
-  )
-  (symbol (lib_id "Device:Crystal_GND24") (at 80.01 127 270) (unit 1)
-    (in_bom yes) (on_board yes) (dnp no)
-    (property "Reference" "Y1" (at 68.58 125.73 90)
-      (effects (font (size 1.27 1.27)) (justify left))
-    )
-    (property "Value" "24MHz" (at 67.31 128.27 90)
-      (effects (font (size 1.27 1.27)) (justify left))
-    )
-    (property "Footprint" "Crystal:Crystal_SMD_SeikoEpson_MC146-4Pin_6.7x1.5mm_HandSoldering" (at 80.01 127 0)
-      (effects (font (size 1.27 1.27)) hide)
-    )
-    (property "Datasheet" "~" (at 80.01 127 0)
-      (effects (font (size 1.27 1.27)) hide)
-    )
-    (pin "1")
-    (pin "2")
-    (pin "3")
-    (pin "4")
-    (instances
-      (project "alarmclock"
-        (path "/fcd099cf-d7c6-418d-b6d0-a7fbd5aabc64"
-          (reference "Y1") (unit 1)
         )
       )
@@
         )
       )
+    )
+  )
+  (symbol (lib_id "Device:Crystal") (at 80.01 128.27 270) (unit 1)
+    (in_bom yes) (on_board yes) (dnp no)
+    (property "Reference" "Y2" (at 72.39 127 90)
+      (effects (font (size 1.27 1.27)) (justify left))
+    )
+    (property "Value" "32.768khz" (at 66.04 129.54 90)
+      (effects (font (size 1.27 1.27)) (justify left))
+    )
+    (property "Footprint" "Crystal:Crystal_SMD_3215-2Pin_3.2x1.5mm" (at 80.01 128.27 0)
+      (effects (font (size 1.27 1.27)) hide)
+    )
+    (property "Datasheet" "~" (at 80.01 128.27 0)
+      (effects (font (size 1.27 1.27)) hide)
+    )
+    (pin "1")
+    (pin "2")
+    (instances
+      (project "alarmclock"
+        (path "/fcd099cf-d7c6-418d-b6d0-a7fbd5aabc64"
+          (reference "Y2") (unit 1)
+        )
+      )

Commit message: tape out
Parts:
- removed C7, C8: 12pF, Capacitor_SMD:C_0805_2012Metric, symbol Device:C_Small
- removed Y2: 32.768khz, Crystal:Crystal_SMD_3215-2Pin_3.2x1.5mm, symbol Device:Crystal
- added F1: Polyfuse, Fuse:Fuse_1206_3216Metric, symbol Device:Polyfuse
- added X2: ECS-327TXO-33-TR, clockcyrstal:ECS-327_ECS, symbol clockcyrstal:ECS-327TXO-33-TR
- JP2: value SolderJumper_BOOT0 -> Jumper_BOOT0
Connections:
- net +5V: now also F1.2; no longer J1.2 (Pin_2)
- net +BATT: now also X2.1 (OUTPUT_ENABLE), X2.4 (SUPPLY)
- net GND: now also X2.2 (GND)
- net OSC_IN: now also X2.3 (OUTPUT)
- net OSC_OUT: no longer names the net of U1.3 (PC15)
- new net: F1.1, J1.2 (Pin_2)
- no-connect marks 5 -> 6
Other:
- note added: "Power input. LDO regulates 5V down to 3,3V. With battery backup and a PMOS that prevents backpowering power hungry devices when using the battery."
- note removed: "Power input. LDO regulates 5V down to 3,3V. With battery backup and a PMOS that prevents backpowering power hungry devices."
- note removed: "kristal uitzoeken"
- moved on the sheet: C1, C2, C3, C4, C5, C6, C9, J1, J3, J4, J6, JP2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
